Commit message: final tested config

File: cohan_navigation/robots/tiago_dual/urdf/tiago_dual.urdf (robot description, URDF)
Before this commit: robot tiago_dual, 70 links, 69 joints
Links:
- link base_link: geometry collision mesh filename=file://../assets/meshes/stl/base_collision.stl scale=1.0 1.0 1.0; visual mesh filename=file://../assets/meshes/stl/base_collision.stl scale=1.0 1.0 1.0
